File: Hardware/Teststand.brd (EAGLE design)
At the start: 94.5 x 65 mm, 69 parts, among them IC1 STM32F103VET, IC2 MAX11254, IC3 MCP2558, IC4 MCP16331, IC5 MCP1700T33, X1 D-SUB25-H3M25RA, X3 MINI-USB_SHIELD4P-85-32004-30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

Commit message: BOM, Gerber + PCB art
Parts:
- removed C13, C14: 10u/100V, rcl:C2220K
- removed C15, C16: 10u, rcl:C1206
- removed C18: 100n, rcl:C0603K
- removed C19: 20p, rcl:C0603K
- removed D1: 4148, diode:SOD123
- removed D2: MBRS1100, diode:SMB
- removed IC4: MCP16331, custom-ic:SOT23-6L
- removed L3: 22u, we-power:L_NR60XX
- removed R26: 52k3, rcl:R0603
- removed R27: 10k, rcl:R0603
- added C22: 1n, rcl:C0603K
- added C23, C26: 1u, rcl:C0603K
- added C24, C25, C27: 10n, rcl:C0603K
- added IC6: AD8538, analog-devices:SO8
- added L1, L4: 600/0.2A (ferrite), rcl:L2012C
- added R30: KELVIN_RC, custom-lcr:CST0612
- added R31, R32: 1k, rcl:R0603
- added R33: 51k, rcl:R0603
- added R34, R35, R41: 100k, rcl:R0603
- added R36: 10k, rcl:R0603
- added V+, V-_IN, V-_OUT: (no value), dmm:4MMJACK
- X3: value MINI-USB_SHIELD4P-85-32004-30X-1 -> MINI-USB_SHIELD4P-85-32004-10X; device con-cypressindustries:85-32004-30X-1 -> con-cypressindustries:85-32004-10X
- moved C20 68.1 mm to (25.9, 9.30)
- moved C21 68.1 mm to (23.8, 9.30)
- moved IC5 68.1 mm to (20.7, 9.30)
- moved C17 67.8 mm to (17.1, 9.30)
- moved X3 29.3 mm to (36.5, 10.2), turned to 90 degrees
- moved R15 20.1 mm to (37.6, 17.9), turned to 270 degrees
- moved R2 19.5 mm to (36.1, 17.9), turned to 270 degrees
- moved R17 2.90 mm to (42.0, 48.6)
- moved R18 2.90 mm to (29.5, 48.6)
- moved R19 2.90 mm to (32.0, 48.6)
- moved R20 2.90 mm to (49.5, 48.6)
- moved R21 2.90 mm to (52.0, 48.6)
- moved R22 2.90 mm to (14.5, 48.6)
- moved R23 2.90 mm to (17.0, 48.6)
- moved R24 2.90 mm to (22.0, 48.6)
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- renumbered JP1 to DBG
Connections:
- removed net SPI3_MISO: IC1.90
- removed net SPI3_MOSI: IC1.91
- removed net SPI3_SCK: IC1.89
- removed net VBAT: IC1.6
- removed net VDDA: IC1.22
- removed net VREF+: IC1.21
- removed net VREF-: IC1.20
- removed net VSSA: IC1.19
- new net ADC_CURRENT: C22.2, IC1.16, IC6.6, R33.2
- new net ADC_VOLTAGE: C25.1, IC1.15, R35.1, R36.2
- new net N$70: R35.2, V+.1@1, V+.1@2
- new net N$71: R30.A, V-_OUT.1@1, V-_OUT.1@2
- new net N$72: C26.1, C27.1, IC1.21, IC1.22, L4.1
- new net N$73: C23.1, C24.1, IC6.4, L1.1, R34.2
- new net N$74: R30.SA, R32.1
- new net N$75: C22.1, IC6.2, R32.2, R33.1
- new net N$76: R30.SB, R31.1
- new net N$77: IC6.3, R31.2, R34.1, R41.2
- net +3V3: now also IC1.6, L1.2, L4.2
- net +5V: now also X3.1; no longer C15.1, C16.1, C19.1, D1.A, L3.2, R26.2
- net GND: now also C23.2, C24.2, C25.2, C26.2, C27.2, IC1.19, IC1.20, IC1.94, IC6.7, R30.B, R36.1, R41.1, V-_IN.1@1, V-_IN.1@2; no longer C13.2, C14.2, C15.2, C16.2, D2.A, IC4.2, R27.2
- net N$55: now also IC1.34, IC2.27; no longer C13.1, C14.1, IC4.5
- net N$65: now also IC1.33, IC2.1; no longer C18.2, D2.C, IC4.6, L3.1
- net N$66: now also IC1.35, IC2.31; no longer C18.1, D1.C, IC4.1
- net N$69: now also IC1.36, X1.12; no longer C19.2, IC4.3, R26.1, R27.1
- net PPM: now also IC1.37
Routing:
- net +5V: track 0.00 -> 163.5 mm, vias 0 -> 10
- net SPI1_SCK: track 2.56 -> 144.1 mm, vias 0 -> 4
- net SPI1_MOSI: track 0.00 -> 126.5 mm, vias 0 -> 3
- net SPI1_MISO: track 0.00 -> 110.4 mm, vias 0 -> 3
- net N$69: track 0.00 -> 52.4 mm, vias 0 -> 2
- net GND: track 29.3 -> 80.8 mm, vias 10 -> 25
- net N$66: track 0.00 -> 41.5 mm, vias 0 -> 2
- net N$65: track 0.00 -> 41.4 mm, vias 0 -> 2
- net N$68: track 0.00 -> 41.3 mm, vias 0 -> 1
- net N$55: track 0.00 -> 39.6 mm, vias 0 -> 2
- net CAN_RX: track 0.00 -> 35.2 mm, vias 0 -> 2
- net N$21: track 0.00 -> 34.0 mm, vias 0 -> 1
- net N$67: track 0.00 -> 32.0 mm, vias 0 -> 1
- net CAN_TX: track 0.00 -> 31.1 mm, vias 0 -> 2
- net N$20: track 0.00 -> 29.9 mm, vias 0 -> 1
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- added copper zone on layer 1, net GND
- added copper zone on layer 1, net N$71
- added copper zone on layer 1, net N$78
Other:
- board text added: "3V3"
- board text added: "5V"
- board text added: "CLK"
- board text added: "DIO"
- board text added: "GND"
- board text added: "H"
- board text added: "L"
- board text added: "MISO"
- board text added: "MOSI"
- board text added: "NSS"
- board text added: "PPM"
- board text added: "RX"
- board text added: "SCK"
- board text added: "SCL"
- board text added: "SDA"
- board text added: "TX"
- board text added: "Teststand V1 01/19"
- board text added: "github.com/jankae/Teststand"
