File: Hardware/Teststand.sch (EAGLE design)
At the start: 69 parts, among them IC1 STM32F103VET, IC2 MAX11254, IC3 MCP2558, IC4 MCP16331, IC5 MCP1700T33, X1 D-SUB25-H3M25RA, X3 MINI-USB_SHIELD4P-85-32004-30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

Commit message: BOM, Gerber + PCB art
Parts:
- removed C13, C14: 10u/100V, rcl:C-EUC2220K
- removed C15, C16: 10u, rcl:C-EUC1206
- removed C18: 100n, rcl:C-EUC0603K
- removed C19: 20p, rcl:C-EUC0603K
- removed D1: 4148, diode:DIODE-SOD123
- removed D2: MBRS1100, diode:DIODE-SMB
- removed IC4: MCP16331, custom-ic:MCP16331
- removed L3: 22u, we-power:INDUCTOR-NR60XX
- removed R26: 52k3, rcl:R-EU_R0603
- removed R27: 10k, rcl:R-EU_R0603
- added C22: 1n, rcl:C-EUC0603K
- added C23, C26: 1u, rcl:C-EUC0603K
- added C24, C25, C27: 10n, rcl:C-EUC0603K
- added IC6: AD8538, analog-devices:AD8519R
- added L1, L4: 600/0.2A (ferrite), rcl:L-EUL2012C
- added R30: KELVIN_RC, custom-lcr:KELVIN_RC
- added R31, R32: 1k, rcl:R-EU_R0603
- added R33: 51k, rcl:R-EU_R0603
- added R34, R35, R41: 100k, rcl:R-EU_R0603
- added R36: 10k, rcl:R-EU_R0603
- added V+, V-_IN, V-_OUT: 4MMJACK, dmm:4MMJACK
- X3: value MINI-USB_SHIELD4P-85-32004-30X-1 -> MINI-USB_SHIELD4P-85-32004-10X; device con-cypressindustries:MINI-USB_SHIELD4P-85-32004-30X-1 -> con-cypressindustries:MINI-USB_SHIELD4P-85-32004-10X
- renumbered JP1 to DBG
Connections:
- removed net SPI3_MISO: IC1MCU.PB4
- removed net SPI3_MOSI: IC1MCU.PB5
- removed net SPI3_SCK: IC1MCU.PB3
- new net ADC_CURRENT: C22.2, IC1MCU.PC1, IC6.OUT, R33.2
- new net ADC_VOLTAGE: C25.1, IC1MCU.PC0, R35.1, R36.2
- new net N$70: R35.2, V+.1, V+.2
- new net N$71: R30.A, V-_OUT.1, V-_OUT.2
- new net N$72: C26.1, C27.1, IC1MCU.VDDA, IC1MCU.VREF+, L4.1
- new net N$73: C23.1, C24.1, IC6.-VS, L1.1, R34.2
- new net N$74: R30.SA, R32.1
- new net N$75: C22.1, IC6.IN-, R32.2, R33.1
- new net N$76: R30.SB, R31.1
- new net N$77: IC6.IN+, R31.2, R34.1, R41.2
- net +3V3: now also IC1MCU.VBAT, L1.2, L4.2
- net +5V: now also X3G$1.1; no longer C15.1, C16.1, C19.1, D1.A, L3.2, R26.2
- net GND: now also C23.2, C24.2, C25.2, C26.2, C27.2, IC1MCU.BOOT0, IC1MCU.VREF-, IC1MCU.VSSA, IC6.+VS, R30.B, R36.1, R41.1, V-_IN.1, V-_IN.2; no longer C13.2, C14.2, C15.2, C16.2, D2.A, IC4.GND, R27.2
- net N$55: now also IC1MCU.PC5, IC2.RSTB; no longer C13.1, C14.1, IC4.VIN
- net N$65: now also IC1MCU.PC4, IC2.RDYB; no longer C18.2, D2.C, IC4.SW, L3.1
- net N$66: now also IC1MCU.PB0, IC2.CSB; no longer C18.1, D1.C, IC4.BOOST
- net N$69: now also IC1MCU.PB1, X1-12.F; no longer C19.2, IC4.FB, R26.1, R27.1
- net PPM: now also IC1MCU.PB2
Other:
- moved on the sheet: C17, C20, C21, IC5
